File: RX.sch (KiCad schematic (older format))
At the start: 14 parts

Commit message: 4 layer add
Parts:
- removed J?: Conn_01x02_Female, Connector_PinHeader_2.54mm:PinHeader_1x02_P2.54mm_Vertical, symbol Connector:Conn_01x02_Female
- added J15: UART4_con, Connector_JST:JST_ZE_SM04B-ZESS-TB_1x04-1MP_P1.50mm_Horizontal, symbol Connector:Conn_01x04_Male
- J11: renamed from J?; footprint Connector_PinHeader_2.54mm:PinHeader_1x04_P2.54mm_Vertical -> Connector_JST:JST_SH_SM04B-SRSS-TB_1x04-1MP_P1.00mm_Horizontal
- J14: renamed from J?; footprint Connector_JST:JST_PH_B4B-PH-SM4-TB_1x04-1MP_P2.00mm_Vertical -> Connector_JST:JST_SH_BM04B-SRSS-TB_1x04-1MP_P1.00mm_Vertical
- J17: renamed from J?; footprint Connector_JST:JST_GH_SM06B-GHS-TB_1x06-1MP_P1.25mm_Horizontal -> Connector_JST:JST_ZE_BM06B-ZESS-TBT_1x06-1MP_P1.50mm_Vertical
- R5: renamed from R?; value 12k -> 10k
- R6: renamed from R?; value 3k -> 10k
- gave numbers to parts that had none: 8
Connections:
- net GND: now also J15.1 (Pin_1)
- net UART1_RX: now also J10.2 (Pin_2); no longer J10.3 (Pin_3)
- net UART1_TX: now also J10.3 (Pin_3); no longer J10.2 (Pin_2)
- net UART5_RX: now also J13.2 (Pin_2); no longer J13.3 (Pin_3)
- net UART5_TX: now also J13.3 (Pin_3); no longer J13.2 (Pin_2)
- net VCC: no longer J13.4 (Pin_4), J14.4 (Pin_4), Rc_sbus2.2
- net +5V: now reaches R5.1
- net +5V: now also J13.4 (Pin_4), J14.4 (Pin_4), Rc_sbus2.2, J15.4 (Pin_4)
- net ADC1 renamed 5V_SENSE
- new net I2C2_SCl: J15.3 (Pin_3)
- new net I2C2_SDA: J15.2 (Pin_2)
- no-connect marks 1 -> 0
Other:
- moved on the sheet: J17, R5, R6
