File: RX.sch (KiCad schematic (older format))
At the start: 15 parts, among them J10 Conn_01x04_Male, J11 Conn_01x04_Male, J12 Conn_01x04_Male, J13 Conn_01x04_Male, J14 UART4_con, J15 UART4_con, J16 UART4_con, J17 Conn_01x06_Male, J9 UART4_con, Q2 2N3904

Commit message: finish board
Parts:
- added J21, J22: Conn_01x06_Male, Connector_JST:JST_SH_SM06B-SRSS-TB_1x06-1MP_P1.00mm_Horizontal, symbol Connector:Conn_01x06_Male
- added J6: Conn_01x04_Male, Connector_JST:JST_SH_SM04B-SRSS-TB_1x04-1MP_P1.00mm_Horizontal, symbol Connector:Conn_01x04_Male
- J14: footprint Connector_JST:JST_SH_BM04B-SRSS-TB_1x04-1MP_P1.00mm_Vertical -> Connector_JST:JST_SH_SM04B-SRSS-TB_1x04-1MP_P1.00mm_Horizontal
Connections:
- net +5V: now also J10.4 (Pin_4), J12.4 (Pin_4), J16.1 (Pin_1), J17.1 (Pin_1), J9.4 (Pin_4), J21.6 (Pin_6), J22.6 (Pin_6), J6.4 (Pin_4)
- net GND: now also J21.1 (Pin_1), J22.1 (Pin_1), J6.1 (Pin_1)
- net I2C2_SCl: now also J15.2 (Pin_2); no longer J15.3 (Pin_3)
- net I2C2_SDA: now also J15.3 (Pin_3); no longer J15.2 (Pin_2)
- net I2C_SCl: now also J14.2 (Pin_2); no longer J14.3 (Pin_3)
- net I2C_SDA: now also J14.3 (Pin_3); no longer J14.2 (Pin_2)
- net UART1_RX: now also J10.3 (Pin_3); no longer J10.2 (Pin_2)
- net UART1_TX: now also J10.2 (Pin_2); no longer J10.3 (Pin_3)
- removed net VCC: J10.4 (Pin_4), J11.4 (Pin_4), J12.4 (Pin_4), J16.1 (Pin_1), J17.1 (Pin_1), J9.4 (Pin_4)
- new net +3V3: J11.4 (Pin_4)
- new net BATT_CURRENT_SENSE: J22.5 (Pin_5)
- new net BATT_VOLT_SENSE: J22.4 (Pin_4)
- new net LED_SAFETY: J22.2 (Pin_2)
- new net SAFETY_SWITCH_IN: J22.3 (Pin_3)
- new net SPI3_CS: J21.5 (Pin_5)
- new net SPI3_MISO: J21.3 (Pin_3)
- new net SPI3_MOSI: J21.2 (Pin_2)
- new net SPI3_SCK: J21.4 (Pin_4)
- new net UART8_RX: J6.2 (Pin_2)
- new net UART8_TX: J6.3 (Pin_3)
