File: _autosave-RX.sch (KiCad schematic (older format))
At the start: 15 parts, among them J10 Conn_01x04_Male, J11 Conn_01x04_Male, J12 Conn_01x04_Male, J13 Conn_01x04_Male, J14 UART4_con, J15 UART4_con, J16 UART4_con, J17 Conn_01x06_Male, J9 UART4_con, Q2 2N3904

Commit message: a
Parts:
- J10: footprint Connector_PinHeader_2.54mm:PinHeader_1x04_P2.54mm_Vertical -> Connector_JST:JST_SH_SM04B-SRSS-TB_1x04-1MP_P1.00mm_Horizontal
- J15: footprint Connector_JST:JST_ZE_SM04B-ZESS-TB_1x04-1MP_P1.50mm_Horizontal -> Connector_JST:JST_SH_SM04B-SRSS-TB_1x04-1MP_P1.00mm_Horizontal
Changed lines of the file:
@@
 F 0 "J10" H 4322 4382 50  0000 R CNN
 F 1 "Conn_01x04_Male" H 4322 4473 50  0001 R CNN
-F 2 "Connector_PinHeader_2.54mm:PinHeader_1x04_P2.54mm_Vertical" H 4350 4500 50  0001 C CNN
+F 2 "Connector_JST:JST_SH_SM04B-SRSS-TB_1x04-1MP_P1.00mm_Horizontal" H 4350 4500 50  0001 C CNN
 F 3 "~" H 4350 4500 50  0001 C CNN
 	1    4350 4500
@@
 F 0 "J15" H 5472 6382 50  0000 R CNN
 F 1 "UART4_con" V 5472 6473 50  0001 R CNN
-F 2 "Connector_JST:JST_ZE_SM04B-ZESS-TB_1x04-1MP_P1.50mm_Horizontal" H 5500 6500 50  0001 C CNN
+F 2 "Connector_JST:JST_SH_SM04B-SRSS-TB_1x04-1MP_P1.00mm_Horizontal" H 5500 6500 50  0001 C CNN
 F 3 "~" H 5500 6500 50  0001 C CNN
 	1    5500 6500
