File: Pixracer_clone.kicad_pcb (KiCad board)
At the start: 4 copper layers, 47.5 x 47.5 mm, 99 parts, among them J1 Conn_01x03_Male, J10 Conn_01x04_Male, J11 Conn_01x04_Male, J12 Conn_01x02_Female, J13 Conn_01x04_Male, J14 UART4_con, J15 UART4_con, J16 UART4_con, J17 Conn_01x06_Male, J18 Micro_SD_Card, J2 USB_B_Micro, J20 Conn_01x04_Male, J3 Conn_01x08_Male, J4 Conn_01x08_Male, J5 Conn_01x08_Male, J6 Conn_01x02_Male, J7 Conn_01x03_Male, J8 Conn_01x02_Male, J9 UART4_con, Q1 2N3904, Q2 2N3904, SW1 SW_Push, U1 STM32F427VITx, U10 LP5907MFX-3.3, U11 NRF24L01_Breakout, U2 USBLC6-2SC6, U3 ICM-20948, U4 MPU-9250, U5 LSM6DS3, U6 TJA1051T, U7 LP5907MFX-1.8, U8 LP5907MFX-3.3, Y1 Crystal_GND24

Commit message: a
Parts:
- removed C18: C, Capacitor_SMD:C_0402_1005Metric
- removed C25: CP, Capacitor_SMD:C_1206_3216Metric
- removed C27: 0.1uF, Capacitor_SMD:C_0603_1608Metric
- removed R4: R, Resistor_SMD:R_0402_1005Metric
- added C15: C, Capacitor_SMD:C_0603_1608Metric, F.Cu at (192.6, 139.3)
- added C42: 0.1uF, Capacitor_SMD:C_0603_1608Metric, F.Cu at (161.9, 114.5)
- added U9: 25LCxxx, Package_SO:SOIC-8-1EP_3.9x4.9mm_P1.27mm_EP2.29x3mm, F.Cu at (180.5, 102.4)
- C1: footprint Capacitor_SMD:C_1206_3216Metric -> Capacitor_SMD:C_0805_2012Metric_Pad1.15x1.40mm_HandSolder
- C17, C19, C23, C24, C26, C29, C31, C32, C33, R3, U3, U4, U5, U7, U8: moved to F.Cu
- C3: footprint Capacitor_SMD:C_1206_3216Metric -> Capacitor_SMD:C_0805_2012Metric
- C7, R5, R6, Rc_sbus1: moved to B.Cu
- J1: footprint Connector_PinHeader_2.54mm:PinHeader_1x03_P2.54mm_Vertical -> Connector_PinHeader_2.54mm:PinHeader_1x03_P2.54mm_Vertical_SMD_Pin1Left
- J10: footprint Connector_PinHeader_2.54mm:PinHeader_1x04_P2.54mm_Vertical -> Connector_JST:JST_SH_SM04B-SRSS-TB_1x04-1MP_P1.00mm_Horizontal; moved to B.Cu
- J12: value Conn_01x02_Female -> Conn_01x04_Male; footprint Connector_PinHeader_2.54mm:PinHeader_1x02_P2.54mm_Vertical -> Connector_JST:JST_SH_SM04B-SRSS-TB_1x04-1MP_P1.00mm_Horizontal
- J15: footprint Connector_JST:JST_ZE_SM04B-ZESS-TB_1x04-1MP_P1.50mm_Horizontal -> Connector_JST:JST_SH_SM04B-SRSS-TB_1x04-1MP_P1.00mm_Horizontal
- J16: footprint Connector_JST:JST_PH_B4B-PH-SM4-TB_1x04-1MP_P2.00mm_Vertical -> Connector_JST:JST_SH_SM04B-SRSS-TB_1x04-1MP_P1.00mm_Horizontal
- J17: footprint Connector_JST:JST_ZE_BM06B-ZESS-TBT_1x06-1MP_P1.50mm_Vertical -> Connector_JST:JST_SH_SM06B-SRSS-TB_1x06-1MP_P1.00mm_Horizontal
- J7: footprint Connector_PinHeader_2.54mm:PinHeader_1x03_P2.54mm_Vertical -> Connector_JST:JST_SH_BM03B-SRSS-TB_1x03-1MP_P1.00mm_Vertical
- moved C34 133.7 mm to (181.3, 97.9), turned to 180 degrees
- moved C22 131.4 mm to (220.2, 98.5), turned to 90 degrees
- moved R6 128.5 mm to (141.4, 140.2)
- moved J6 120.5 mm to (188.4, 88.8), turned to 90 degrees
- moved R5 114.7 mm to (145.0, 140.2)
- moved D6 97.8 mm to (202.0, 78.5)
- moved R10 96.1 mm to (202.0, 80.0)
- moved C28 93.4 mm to (181.7, 116.8), turned to 270 degrees
- moved C36 92.8 mm to (200.4, 86.2)
- moved C37 92.8 mm to (200.4, 87.8)
- moved R2 89.9 mm to (156.6, 85.1), turned to 90 degrees
- moved J12 86.3 mm to (148.7, 111.8), turned to 270 degrees
- moved Q1 82.7 mm to (152.8, 85.2), turned to 180 degrees
- moved J9 81.5 mm to (200.2, 64.4), turned to 0 degrees
- moved C16 81.2 mm to (170.1, 114.8), turned to 270 degrees
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Connections:
- J12 pad 1: Net-(J12-Pad1) -> GND
- J12 pad 2: GND -> UART7_RX
- J3 pad 1: TIM3_CH1 -> TIM3_CH4
- J3 pad 2: TIM3_CH2 -> TIM3_CH3
- J3 pad 3: TIM3_CH3 -> TIM3_CH2
- J3 pad 4: TIM3_CH4 -> TIM3_CH1
- U1 pad 51: EXTERNAL_MEM_CS -> Net-(U1-Pad51)
- U1 pad 57: Net-(U1-Pad57) -> EXTERNAL_MEM_CS
Routing:
- net GND: track 26.5 -> 72.7 mm, vias 21 -> 24
- net IMU_MOSI: track 2.88 -> 31.3 mm, vias 1 -> 5
- net +3.3VA: track 0.00 -> 28.3 mm, vias 2 -> 3
- net TIM1_CH3: track 0.00 -> 24.7 mm
- net TIM1_CH4: track 0.00 -> 24.2 mm
- net +1V8: track 0.00 -> 22.9 mm, vias 0 -> 3
- net TIM1_CH1: track 0.00 -> 22.2 mm
- net TIM1_CH2: track 0.00 -> 22.0 mm
- net IMU_MISO: track 9.17 -> 27.0 mm, vias 1 -> 3
- net EXTERNAL_MEM_CS: track 0.00 -> 13.6 mm
- net VCC: track 1.84 -> 15.1 mm
- net TIM3_CH4: track 0.00 -> 13.2 mm
- net LSM6D3_CS: track 3.70 -> 15.5 mm, vias 1 -> 2
- net TIM3_CH1: track 0.00 -> 11.6 mm
- net TIM3_CH3: track 0.00 -> 11.6 mm
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Other:
- outline, holes or cut-outs redrawn
