File: Pixracer_clone.kicad_pcb (KiCad board)
At the start: 4 copper layers, 47.5 x 47.5 mm, 99 parts, among them J1 Conn_01x03_Male, J10 Conn_01x04_Male, J11 Conn_01x04_Male, J12 Conn_01x02_Female, J13 Conn_01x04_Male, J14 UART4_con, J15 UART4_con, J16 UART4_con, J17 Conn_01x06_Male, J18 Micro_SD_Card, J2 USB_B_Micro, J20 Conn_01x04_Male, J3 Conn_01x08_Male, J4 Conn_01x08_Male, J5 Conn_01x08_Male, J6 Conn_01x02_Male, J7 Conn_01x03_Male, J8 Conn_01x02_Male, J9 UART4_con, Q1 2N3904, Q2 2N3904, SW1 SW_Push, U1 STM32F427VITx, U10 LP5907MFX-3.3, U11 NRF24L01_Breakout, U2 USBLC6-2SC6, U3 ICM-20948, U4 MPU-9250, U5 LSM6DS3, U6 TJA1051T, U7 LP5907MFX-1.8, U8 LP5907MFX-3.3, Y1 Crystal_GND24

Commit message: add alittle
Parts:
- moved C31 82.2 mm to (170.7, 110.4), turned to 90 degrees
- moved C17 64.7 mm to (160.3, 109.0), turned to 180 degrees
- moved C10 47.5 mm to (182.9, 62.8)
- moved C11 47.5 mm to (185.8, 64.7)
- moved C12 47.5 mm to (188.7, 62.3)
- moved C5 47.5 mm to (182.9, 64.7)
- moved C6 47.5 mm to (185.8, 62.8)
- moved J12 16.7 mm to (81.4, 57.9)
- moved J10 5.60 mm to (157.8, 131.2)
- moved J13 5.60 mm to (157.8, 128.1)
- moved J9 5.60 mm to (157.7, 134.0)
- moved Q2 2.24 mm to (154.3, 104.6)
- moved Rc_sbus2 2.24 mm to (151.8, 104.6)
- moved Rb_sbus1 2.24 mm to (157.3, 104.5)
- moved Rc_sbus1 2.24 mm to (156.4, 107.2)
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Connections:
- U1 pad 24: USART4_RX -> SBUS
Routing:
- net GND: track 2.16 -> 26.5 mm, vias 14 -> 23
- net USB_D-: track 0.00 -> 19.1 mm
- net USB_D+: track 0.00 -> 19.1 mm
- net SDIO3: track 1.61 -> 17.4 mm, vias 0 -> 1
- net SDIO_CLK: track 8.35 -> 23.9 mm
- net SDIO_CMD: track 8.39 -> 17.9 mm
- net OSC1+: track 0.00 -> 7.51 mm
- net OSC1-: track 0.00 -> 5.30 mm
- net Net-(C2-Pad1): track 0.00 -> 1.93 mm
- net SDIO2: track 13.5 -> 15.0 mm, vias 0 -> 1
- net SDIO0: track 27.3 -> 26.3 mm
- removed copper zone on In1.Cu, net GND
- removed copper zone on In2.Cu, net GND
Other:
- net class OSC added: clearance 0.15, trace_width 0.25, via_dia 0.6, via_drill 0.3

Commit message: add alot
Parts:
- C17, C18, C19, C23, C24, C25, C26, C27, C29, C31, C32, C33, R3, U3, U4, U5, U7, U8: moved to B.Cu
- moved C25 87.1 mm to (158.3, 116.5), turned to 90 degrees
- moved C33 83.3 mm to (174.5, 115.2), turned to 90 degrees
- moved C19 80.0 mm to (172.1, 114.3)
- moved C24 73.9 mm to (163.9, 113.5), turned to 180 degrees
- moved C26 73.8 mm to (160.2, 117.1), turned to 270 degrees
- moved R3 72.1 mm to (171.8, 107.8), turned to 180 degrees
- moved C23 72.0 mm to (161.8, 110.4), turned to 90 degrees
- moved J17 64.8 mm to (233.1, 72.0)
- moved J15 41.5 mm to (216.1, 133.8)
- moved C18 13.3 mm to (175.5, 115.2)
- moved R11 11.5 mm to (165.9, 92.2)
- moved R12 11.5 mm to (164.6, 92.2)
- moved J16 11.5 mm to (181.9, 127.8)
- moved R13 11.5 mm to (167.9, 92.2)
- moved R15 11.5 mm to (171.3, 92.2)
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Connections:
- U1 pad 68: UART1_TX -> Net-(U1-Pad68)
- U1 pad 69: UART1_RX -> Net-(U1-Pad69)
Routing:
- net SWDIO: track 0.00 -> 20.2 mm
- net SDIO_CLK: track 23.9 -> 7.87 mm
- net SWCLK: track 0.00 -> 15.6 mm
- net SDIO3: track 17.4 -> 4.92 mm
- net SDIO_CMD: track 17.9 -> 5.45 mm
- net SDIO0: track 26.3 -> 15.3 mm, vias 1 -> 2
- net SDIO1: track 26.8 -> 15.9 mm
- net SDIO2: track 15.0 -> 4.61 mm
- net MPU9250_CS: track 0.00 -> 6.70 mm, vias 0 -> 2
- net IMU_MISO: track 5.19 -> 9.17 mm, vias 0 -> 1
- net LSM6D3_CS: track 0.00 -> 3.70 mm, vias 0 -> 1
- net IMU_CLK: track 12.9 -> 9.45 mm, vias 0 -> 1
- net IMU_MOSI: track 0.00 -> 2.88 mm, vias 0 -> 1
- net MPU9250_DRDY: track 0.00 -> 2.50 mm, vias 0 -> 1
- net GND: vias 23 -> 21
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
Commit message: a
Parts:
- removed C18: C, Capacitor_SMD:C_0402_1005Metric
- removed C25: CP, Capacitor_SMD:C_1206_3216Metric
- removed C27: 0.1uF, Capacitor_SMD:C_0603_1608Metric
- removed R4: R, Resistor_SMD:R_0402_1005Metric
- added C15: C, Capacitor_SMD:C_0603_1608Metric, F.Cu at (192.6, 139.3)
- added C42: 0.1uF, Capacitor_SMD:C_0603_1608Metric, B.Cu at (163.8, 128.5)
- added U9: 25LCxxx, Package_SO:SOIC-8-1EP_3.9x4.9mm_P1.27mm_EP2.29x3mm, F.Cu at (180.5, 102.4)
- C1: footprint Capacitor_SMD:C_1206_3216Metric -> Capacitor_SMD:C_0805_2012Metric_Pad1.15x1.40mm_HandSolder
- C16, C20, C28, C7, R5, R6, Rc_sbus1: moved to B.Cu
- C3: footprint Capacitor_SMD:C_1206_3216Metric -> Capacitor_SMD:C_0805_2012Metric
- C32, C33, R3: moved to F.Cu
- J1: footprint Connector_PinHeader_2.54mm:PinHeader_1x03_P2.54mm_Vertical -> Connector_PinHeader_2.54mm:PinHeader_1x03_P2.54mm_Vertical_SMD_Pin1Left
- J10: footprint Connector_PinHeader_2.54mm:PinHeader_1x04_P2.54mm_Vertical -> Connector_JST:JST_SH_SM04B-SRSS-TB_1x04-1MP_P1.00mm_Horizontal; moved to B.Cu
- J12: value Conn_01x02_Female -> Conn_01x04_Male; footprint Connector_PinHeader_2.54mm:PinHeader_1x02_P2.54mm_Vertical -> Connector_JST:JST_SH_SM04B-SRSS-TB_1x04-1MP_P1.00mm_Horizontal
- J15: footprint Connector_JST:JST_ZE_SM04B-ZESS-TB_1x04-1MP_P1.50mm_Horizontal -> Connector_JST:JST_SH_SM04B-SRSS-TB_1x04-1MP_P1.00mm_Horizontal
- J16: footprint Connector_JST:JST_PH_B4B-PH-SM4-TB_1x04-1MP_P2.00mm_Vertical -> Connector_JST:JST_SH_SM04B-SRSS-TB_1x04-1MP_P1.00mm_Horizontal
- J17: footprint Connector_JST:JST_ZE_BM06B-ZESS-TBT_1x06-1MP_P1.50mm_Vertical -> Connector_JST:JST_SH_SM06B-SRSS-TB_1x06-1MP_P1.00mm_Horizontal
- J7: footprint Connector_PinHeader_2.54mm:PinHeader_1x03_P2.54mm_Vertical -> Connector_JST:JST_SH_BM03B-SRSS-TB_1x03-1MP_P1.00mm_Vertical
- moved C34 133.7 mm to (181.3, 97.9), turned to 180 degrees
- moved C22 131.4 mm to (220.2, 98.5), turned to 90 degrees
- moved R6 128.5 mm to (141.4, 140.2)
- moved J6 120.5 mm to (188.4, 88.8), turned to 90 degrees
- moved R5 114.7 mm to (145.0, 140.2)
- moved C28 109.1 mm to (193.4, 127.3), turned to 90 degrees
- moved D6 97.8 mm to (202.0, 78.5)
- moved R10 96.1 mm to (202.0, 80.0)
- moved C20 93.7 mm to (176.4, 131.6), turned to 270 degrees
- moved C36 92.8 mm to (200.4, 86.2)
- moved C37 92.8 mm to (200.4, 87.8)
- moved C16 91.9 mm to (172.0, 128.2), turned to 90 degrees
- moved R2 89.9 mm to (156.6, 85.1), turned to 90 degrees
- moved J12 86.3 mm to (148.7, 111.8), turned to 270 degrees
- moved Q1 82.7 mm to (152.8, 85.2), turned to 180 degrees
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Connections:
- J12 pad 1: Net-(J12-Pad1) -> GND
- J12 pad 2: GND -> UART7_RX
- J3 pad 1: TIM3_CH1 -> TIM3_CH4
- J3 pad 2: TIM3_CH2 -> TIM3_CH3
- J3 pad 3: TIM3_CH3 -> TIM3_CH2
- J3 pad 4: TIM3_CH4 -> TIM3_CH1
- U1 pad 51: EXTERNAL_MEM_CS -> Net-(U1-Pad51)
- U1 pad 57: Net-(U1-Pad57) -> EXTERNAL_MEM_CS
Routing:
- net GND: track 26.5 -> 72.7 mm, vias 21 -> 24
- net +3.3VA: track 0.00 -> 28.3 mm, vias 2 -> 3
- net IMU_MOSI: track 2.88 -> 30.8 mm, vias 1 -> 4
- net +1V8: track 0.00 -> 21.7 mm, vias 0 -> 3
- net IMU_MISO: track 9.17 -> 26.7 mm, vias 1 -> 3
- net IMU_CLK: track 9.45 -> 26.6 mm, vias 1 -> 3
- net ICM20948_DRDY: track 0.00 -> 14.0 mm, vias 0 -> 3
- net EXTERNAL_MEM_CS: track 0.00 -> 13.6 mm
- net VCC: track 1.84 -> 15.1 mm
- net TIM3_CH4: track 0.00 -> 13.2 mm
- net TIM3_CH1: track 0.00 -> 11.6 mm
- net TIM3_CH3: track 0.00 -> 11.6 mm
- net LSM6D3_CS: track 3.70 -> 14.5 mm
- net TIM3_CH2: track 0.00 -> 10.7 mm
- net MPU9250_DRDY: track 2.50 -> 12.9 mm, vias 1 -> 2
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Other:
- outline, holes or cut-outs redrawn

Commit message: finish board
Parts:
- removed C11: 1u, Capacitor_SMD:C_0402_1005Metric
- removed C22: CP, Capacitor_SMD:C_1206_3216Metric
- removed C32: 1uF, Capacitor_SMD:C_0402_1005Metric
- removed C33: 100nF, Capacitor_SMD:C_0402_1005Metric
- removed C41: C, Capacitor_SMD:C_0603_1608Metric
- removed F1: Fuse, Fuse:Fuse_1812_4532Metric
- removed J11: Conn_01x04_Male, Connector_JST:JST_SH_SM04B-SRSS-TB_1x04-1MP_P1.00mm_Horizontal
- removed J13: Conn_01x04_Male, Connector_PinHeader_2.54mm:PinHeader_1x04_P2.54mm_Vertical
- removed J14: UART4_con, Connector_JST:JST_SH_BM04B-SRSS-TB_1x04-1MP_P1.00mm_Vertical
- removed J6: Conn_01x02_Male, Connector_PinHeader_2.54mm:PinHeader_1x02_P2.54mm_Vertical
- removed J7: Conn_01x03_Male, Connector_JST:JST_SH_BM03B-SRSS-TB_1x03-1MP_P1.00mm_Vertical
- removed J9: UART4_con, Connector_PinHeader_2.54mm:PinHeader_1x04_P2.54mm_Vertical
- added C25: CP, Capacitor_SMD:C_1206_3216Metric, F.Cu at (179.1, 112.7)
- added C43: 1uF, Capacitor_SMD:C_0603_1608Metric_Pad1.05x0.95mm_HandSolder, F.Cu at (147.8, 85.1)
- added G***: LOGO, pusheen:pusheen_small, F.Cu at (157.9, 86.3)
- added G***: LOGO, Pixracer_clone:pusheen, B.Cu at (166.4, 104.4)
- added I2C1: UART4_con, Connector_JST:JST_SH_SM04B-SRSS-TB_1x04-1MP_P1.00mm_Horizontal, F.Cu at (170.0, 75.5)
- added IMU_Debug: Conn_01x10_Male, Connector_PinHeader_2.54mm:PinHeader_1x10_P2.54mm_Vertical, F.Cu at (157.6, 120.1)
- added J19: Conn_01x02_Male, Connector_PinHeader_2.54mm:PinHeader_1x02_P2.54mm_Vertical, F.Cu at (189.6, 88.2)
- added R4: 22R, Resistor_SMD:R_0603_1608Metric_Pad1.05x0.95mm_HandSolder, F.Cu at (185.9, 82.9)
- added SBUS: Conn_01x04_Male, Connector_JST:JST_SH_SM04B-SRSS-TB_1x04-1MP_P1.00mm_Horizontal, F.Cu at (147.5, 104.4)
- added SPI3: Conn_01x06_Male, Connector_JST:JST_SH_SM06B-SRSS-TB_1x06-1MP_P1.00mm_Horizontal, B.Cu at (147.1, 82.0)
- added SWD: Conn_01x04_Male, Connector_JST:JST_SH_SM04B-SRSS-TB_1x04-1MP_P1.00mm_Horizontal, F.Cu at (185.6, 75.4)
- added Switch: Conn_01x06_Male, Connector_JST:JST_SH_SM06B-SRSS-TB_1x06-1MP_P1.00mm_Horizontal, F.Cu at (147.5, 112.7)
- added UART8: Conn_01x04_Male, Connector_JST:JST_SH_SM04B-SRSS-TB_1x04-1MP_P1.00mm_Horizontal, F.Cu at (162.2, 75.4)
- added x: indicator, Pixracer_clone:indicator, F.Cu at (159.3, 115.9)
- Buzzer: renamed from J8; moved to B.Cu
- C15: value C -> 1uF; footprint Capacitor_SMD:C_0603_1608Metric -> Capacitor_SMD:C_0603_1608Metric_Pad1.05x0.95mm_HandSolder
- C16, C17, C19, C20, C23, C24, C26, C28, C29, C31, C42, C7, R5, R6, Rc_sbus1, U7, U8: moved to F.Cu
- C39, D2, Q1, R2: moved to B.Cu
- I2C2: renamed from J15; moved to F.Cu
- ICM20948: renamed from U3; moved to F.Cu
- LSM6D: renamed from U5; moved to F.Cu
- MPU9250: renamed from U4; moved to F.Cu
- R3: value R -> 22R; footprint Resistor_SMD:R_0402_1005Metric -> Resistor_SMD:R_0603_1608Metric_Pad1.05x0.95mm_HandSolder
- U2: value USBLC6-2SC6 -> LP5907MFX-3.3; footprint Package_TO_SOT_SMD:SOT-23-6 -> Package_TO_SOT_SMD:SOT-23-5
- moved C15 67.0 mm to (153.2, 85.1), turned to 90 degrees
- moved R3 55.7 mm to (185.9, 81.2), turned to 180 degrees
- moved C12 48.5 mm to (157.5, 99.4), turned to 90 degrees
- moved C30 41.9 mm to (185.2, 112.7), turned to 90 degrees
- moved Buzzer 39.6 mm to (186.2, 75.8), turned to 90 degrees
- moved C10 39.5 mm to (157.3, 95.6), turned to 90 degrees
- moved C6 39.0 mm to (156.4, 91.8), turned to 90 degrees
- moved Rc_sbus1 38.4 mm to (156.3, 106.9)
- moved U2 34.8 mm to (150.5, 85.2)
- moved UART3 33.2 mm to (190.7, 113.9), turned to 90 degrees
- moved R6 32.8 mm to (156.3, 111.1)
- moved Q1 31.8 mm to (184.0, 79.3)
- moved R2 31.6 mm to (187.7, 79.4)
- moved R5 29.8 mm to (156.3, 112.6), turned to 180 degrees
- moved C5 29.2 mm to (161.7, 88.0)
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- renumbered J1 to Boot, J20 to CAN, U9 to Memory, J18 to SDcard, U1 to STM32F427VIT6, U6 to TJA1015, J17 to Telemetry, J10 to UART1, J16 to UART3, J12 to UART7, U11 to nRF24
Connections:
- Buzzer pad 2: 5V_IN -> +5V
- C15 pad 1: VBUS -> +5V
- C21 pad 1: 5V_IN -> +5V
- C30 pad 1: 5V_IN -> +5V
- CAN pad 4: 5V_IN -> +5V
- D2 pad 1: 5V_IN -> +5V
- I2C2 pad 2: I2C2_SDA -> I2C2_SCl
- I2C2 pad 3: I2C2_SCl -> I2C2_SDA
- I2C2 pad 4: 5V_IN -> +5V
- J5 pad 1: 5V_IN -> +5V
- J5 pad 2: 5V_IN -> +5V
- J5 pad 3: 5V_IN -> +5V
- J5 pad 4: 5V_IN -> +5V
- J5 pad 5: 5V_IN -> +5V
- J5 pad 6: 5V_IN -> +5V
- J5 pad 7: 5V_IN -> +5V
- J5 pad 8: 5V_IN -> +5V
- R3 pad 1: +3.3VA -> /USB_sheet/D+
- R3 pad 2: ICM20948_CS -> USB_D+
- R5 pad 1: 5V_IN -> +5V
- Rc_sbus2 pad 2: 5V_IN -> +5V
- STM32F427VIT6 pad 3: SPI4_MOSI -> SPI4_CS
- STM32F427VIT6 pad 43: Net-(U1-Pad43) -> EXTERNAL_MPU_CS
- STM32F427VIT6 pad 51: Net-(U1-Pad51) -> EXTERNAL_MEM_CS
- STM32F427VIT6 pad 57: EXTERNAL_MEM_CS -> Net-(U1-Pad57)
- TJA1015 pad 3: 5V_IN -> +5V
- Telemetry pad 1: VCC -> +5V
- U2 pad 1: /USB_sheet/D- -> +5V
- U2 pad 3: /USB_sheet/D+ -> nRF24_EN
- U2 pad 4: USB_D+ -> Net-(U2-Pad4)
- U2 pad 5: VBUS -> Net-(C43-Pad1)
- U8 pad 1: 5V_IN -> +5V
- UART1 pad 2: UART1_RX -> UART1_TX
- UART1 pad 3: UART1_TX -> UART1_RX
- UART1 pad 4: VCC -> +5V
- UART3 pad 1: VCC -> +5V
- UART7 pad 4: VCC -> +5V
- nRF24 pad 1: Net-(U11-Pad1) -> GND
- nRF24 pad 2: Net-(U11-Pad2) -> Net-(C43-Pad1)
- nRF24 pad 3: Net-(U11-Pad3) -> SPI4_CE
- nRF24 pad 4: Net-(U11-Pad4) -> SPI4_CS
- nRF24 pad 5: Net-(U11-Pad5) -> SPI4_CLK
- nRF24 pad 6: Net-(U11-Pad6) -> SPI4_MOSI
- nRF24 pad 7: Net-(U11-Pad7) -> SPI4_MISO
Routing:
- net +5V: track 0.00 -> 215.8 mm, vias 0 -> 19
- net VCC: track 15.1 -> 156.1 mm, vias 4 -> 19
- net GND: track 72.7 -> 140.7 mm, vias 24 -> 77
- net 3.3_SENSE_EN: track 0.00 -> 30.0 mm, vias 0 -> 2
- net UART7_RX: track 0.00 -> 27.7 mm, vias 0 -> 2
- net UART7_TX: track 0.00 -> 27.4 mm, vias 0 -> 2
- net I2C2_SCl: track 0.00 -> 26.2 mm, vias 0 -> 2
- net UART3_TX: track 0.00 -> 26.2 mm, vias 0 -> 2
- net I2C2_SDA: track 0.00 -> 25.0 mm, vias 0 -> 2
- net SPI3_CS: track 0.00 -> 24.3 mm, vias 0 -> 1
- net Buzzer: track 0.00 -> 24.1 mm, vias 0 -> 1
- net nRF24_EN: track 0.00 -> 23.5 mm, vias 0 -> 2
- net SPI3_SCK: track 0.00 -> 23.1 mm, vias 0 -> 1
- net SPI4_MOSI: track 0.00 -> 23.0 mm, vias 0 -> 2
- net UART3_RX: track 0.00 -> 23.0 mm, vias 0 -> 2
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- added copper zone on B.Cu, net GND
- added copper zone on F.Cu, net GND
- added copper zone on In1.Cu, net GND
- added copper zone on In2.Cu, net VCC
Other:
- board size 47.5 x 47.5 mm -> 49.5 x 49.4 mm
- net class Default removed
- net class OSC removed
