File: IMU_board/IMU_board.kicad_pcb (KiCad board)
At the start: 4 copper layers, 28.5 x 26.2 mm, 38 parts, among them J1 Conn_01x10_Male, Q3 BSS138, Q4 BSS138, Q5 BSS138, Q6 BSS138, Q7 BSS138, U3 LP5907MFX-3.3, U4 LSM6DS3, U7 LP5907MFX-1.8

Commit message: add led
Parts:
- added D1: LED, LED_SMD:LED_0603_1608Metric_Pad1.05x0.95mm_HandSolder, F.Cu at (149.5, 103.6)
- added R1: R, Resistor_SMD:R_0603_1608Metric_Pad1.05x0.95mm_HandSolder, F.Cu at (149.6, 105.2)
- renumbered ICM20948 to U1, MPU9250 to U2
Connections:
- U1 pad 1: (no net) -> Net-(U1-Pad1)
- U1 pad 14: (no net) -> Net-(U1-Pad14)
- U1 pad 15: (no net) -> Net-(U1-Pad15)
- U1 pad 16: (no net) -> Net-(U1-Pad16)
- U1 pad 17: (no net) -> Net-(U1-Pad17)
- U1 pad 19: (no net) -> Net-(U1-Pad19)
- U1 pad 2: (no net) -> Net-(U1-Pad2)
- U1 pad 21: (no net) -> Net-(U1-Pad21)
- U1 pad 3: (no net) -> Net-(U1-Pad3)
- U1 pad 4: (no net) -> Net-(U1-Pad4)
- U1 pad 5: (no net) -> Net-(U1-Pad5)
- U1 pad 6: (no net) -> Net-(U1-Pad6)
- U1 pad 7: (no net) -> Net-(U1-Pad7)
- U2 pad 12: (no net) -> MPU9250_DRDY
- U2 pad 21: (no net) -> Net-(U2-Pad21)
- U2 pad 7: (no net) -> Net-(U2-Pad7)
Routing:
- net +3V3: vias 11 -> 12
- removed copper zone on B.Cu, net GND
- removed copper zone on F.Cu, net GND
