File: IMU_board/IMU_board.kicad_sch (KiCad schematic)
At the start: 38 parts, among them J1 Conn_01x10_Male, Q3 BSS138, Q4 BSS138, Q5 BSS138, Q6 BSS138, Q7 BSS138, U1 ICM-20948, U2 MPU-9250, U3 LP5907MFX-3.3, U4 LSM6DS3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

Commit message: add led
Parts:
- added D1: LED, LED_SMD:LED_0603_1608Metric_Pad1.05x0.95mm_HandSolder, symbol Device:LED
- added R1: R, Resistor_SMD:R_0603_1608Metric_Pad1.05x0.95mm_HandSolder, symbol Device:R
Connections:
- net +3V3: now also D1.2 (A)
- net GND: now also R1.2
- new net LED: D1.1 (K), R1.1
Changed lines of the file:
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@@
   (junction (at 254.5588 80.4164) (diameter 1.016) (color 0 0 0 0))
   (junction (at 260.6548 140.2588) (diameter 1.016) (color 0 0 0 0))
+  (junction (at 262.128 51.562) (diameter 1.016) (color 0 0 0 0))
   (no_connect (at 71.12 63.5))
+  (no_connect (at 71.12 60.96))
   (no_connect (at 100.33 134.62))
-  (no_connect (at 71.12 60.96))
   (no_connect (at 100.33 137.16))
   (wire (pts (xy 35.56 71.12) (xy 45.72 71.12))
@@
     (stroke (width 0) (type solid) (color 0 0 0 0))
   )
-  (wire (pts (xy 46.99 138.43) (xy 48.26 138.43))
+  (wire (pts (xy 46.99 138.43) (xy 50.8 138.43))
     (stroke (width 0) (type solid) (color 0 0 0 0))
   )
@@
     (stroke (width 0) (type solid) (color 0 0 0 0))
   )
-  (wire (pts (xy 50.8 138.43) (xy 48.26 138.43))
-    (stroke (width 0) (type solid) (color 0 0 0 0))
-  )
   (wire (pts (xy 55.88 43.18) (xy 55.88 41.91))
     (stroke (width 0) (type solid) (color 0 0 0 0))
@@
     (stroke (width 0) (type solid) (color 0 0 0 0))
   )
-  (wire (pts (xy 60.96 43.18) (xy 60.96 45.72))
-    (stroke (width 0) (type solid) (color 0 0 0 0))
-  )
   (wire (pts (xy 60.96 137.16) (xy 64.77 137.16))
     (stroke (width 0) (type solid) (color 0 0 0 0))
@@
     (stroke (width 0) (type solid) (color 0 0 0 0))
   )
-  (wire (pts (xy 81.534 106.68) (xy 81.28 106.68))
-    (stroke (width 0) (type solid) (color 0 0 0 0))
-  )
   (wire (pts (xy 82.55 160.02) (xy 82.55 168.91))
     (stroke (width 0) (type solid) (color 0 0 0 0))
@@
     (stroke (width 0) (type solid) (color 0 0 0 0))
   )
+  (wire (pts (xy 258.1148 51.562) (xy 258.1148 51.3588))
+    (stroke (width 0) (type solid) (color 0 0 0 0))
+  )
   (wire (pts (xy 258.6736 140.2588) (xy 260.6548 140.2588))
     (stroke (width 0) (type solid) (color 0 0 0 0))
@@
   )
   (wire (pts (xy 260.6548 140.2588) (xy 263.398 140.2588))
+    (stroke (width 0) (type solid) (color 0 0 0 0))
+  )
+  (wire (pts (xy 262.0772 37.4396) (xy 261.874 37.4396))
+    (stroke (width 0) (type solid) (color 0 0 0 0))
+  )
+  (wire (pts (xy 262.0772 42.7228) (xy 262.0772 37.4396))
+    (stroke (width 0) (type solid) (color 0 0 0 0))
+  )
+  (wire (pts (xy 262.128 50.3428) (xy 262.0772 50.3428))
+    (stroke (width 0) (type solid) (color 0 0 0 0))
+  )
+  (wire (pts (xy 262.128 51.562) (xy 258.1148 51.562))
+    (stroke (width 0) (type solid) (color 0 0 0 0))
+  )
+  (wire (pts (xy 262.128 51.562) (xy 262.128 50.3428))
+    (stroke (width 0) (type solid) (color 0 0 0 0))
+  )
+  (wire (pts (xy 262.128 59.182) (xy 262.128 62.6364))
     (stroke (width 0) (type solid) (color 0 0 0 0))
   )
@@
     (effects (font (size 1.27 1.27)) (justify right))
   )
+  (global_label "LED" (shape input) (at 258.1148 51.3588 180)
+    (effects (font (size 1.27 1.27)) (justify right))
+  )
   (global_label "IMU_MOSI_3.3v" (shape input) (at 263.398 140.2588 0)
     (effects (font (size 1.27 1.27)) (justify left))
@@
     )
   )
+  (symbol (lib_id "power:+3V3") (at 261.874 37.4396 0) (unit 1)
+    (in_bom yes) (on_board yes)
+    (property "Reference" "#PWR0134" (id 0) (at 261.874 41.2496 0)
+      (effects (font (size 1.27 1.27)) hide)
+    )
+    (property "Value" "+3V3" (id 1) (at 262.2423 33.1152 0))
+    (property "Footprint" "" (id 2) (at 261.874 37.4396 0)
+      (effects (font (size 1.27 1.27)) hide)
+    )
+    (property "Datasheet" "" (id 3) (at 261.874 37.4396 0)
+      (effects (font (size 1.27 1.27)) hide)
+    )
+  )
   (symbol (lib_id "power:GND") (at 45.72 43.18 270) (unit 1)
     (in_bom yes) (on_board yes)
@@
     )
   )
+  (symbol (lib_id "power:GND") (at 262.128 62.6364 0) (unit 1)
+    (in_bom yes) (on_board yes)
+    (property "Reference" "#PWR0136" (id 0) (at 262.128 68.9864 0)
+      (effects (font (size 1.27 1.27)) hide)
+    )
+    (property "Value" "GND" (id 1) (at 262.2423 66.9608 0))
+    (property "Footprint" "" (id 2) (at 262.128 62.6364 0)
+      (effects (font (size 1.27 1.27)) hide)
+    )
+    (property "Datasheet" "" (id 3) (at 262.128 62.6364 0)
+      (effects (font (size 1.27 1.27)) hide)
+    )
+  )
   (symbol (lib_id "Device:R") (at 116.7384 182.4228 0) (unit 1)
     (in_bom yes) (on_board yes)
@@
     )
     (property "Datasheet" "~" (id 3) (at 260.6548 133.5532 0)
+      (effects (font (size 1.27 1.27)) hide)
+    )
+  )
+  (symbol (lib_id "Device:R") (at 262.128 55.372 0) (unit 1)
+    (in_bom yes) (on_board yes)
+    (property "Reference" "R1" (id 0) (at 263.9061 54.2226 0)
+      (effects (font (size 1.27 1.27)) (justify left))
+    )
+    (property "Value" "R" (id 1) (at 263.9061 56.5213 0)
+      (effects (font (size 1.27 1.27)) (justify left))
+    )
+    (property "Footprint" "Resistor_SMD:R_0603_1608Metric_Pad1.05x0.95mm_HandSolder" (id 2) (at 260.35 55.372 90)
+      (effects (font (size 1.27 1.27)) hide)
+    )
+    (property "Datasheet" "~" (id 3) (at 262.128 55.372 0)
+      (effects (font (size 1.27 1.27)) hide)
+    )
+  )
+  (symbol (lib_id "Device:LED") (at 262.0772 46.5328 90) (unit 1)
+    (in_bom yes) (on_board yes)
+    (property "Reference" "D1" (id 0) (at 264.9983 45.5739 90)
+      (effects (font (size 1.27 1.27)) (justify right))
+    )
+    (property "Value" "LED" (id 1) (at 264.9983 47.8726 90)
+      (effects (font (size 1.27 1.27)) (justify right))
+    )
+    (property "Footprint" "LED_SMD:LED_0603_1608Metric_Pad1.05x0.95mm_HandSolder" (id 2) (at 262.0772 46.5328 0)
+      (effects (font (size 1.27 1.27)) hide)
+    )
+    (property "Datasheet" "~" (id 3) (at 262.0772 46.5328 0)
       (effects (font (size 1.27 1.27)) hide)
     )
@@
       (reference "#PWR0133") (unit 1) (value "+3V3") (footprint "")
     )
+    (path "/615427c9-94ee-4bb7-b6fc-46a27d7c852f"
+      (reference "#PWR0134") (unit 1) (value "+3V3") (footprint "")
+    )
     (path "/93bcebbc-1fee-4233-9fca-4871aa8a2e97"
       (reference "#PWR0135") (unit 1) (value "+1V8") (footprint "")
     )
+    (path "/f60fc88a-a6a2-4fbb-8ff0-47a2a59583bd"
+      (reference "#PWR0136") (unit 1) (value "GND") (footprint "")
+    )
     (path "/00000000-0000-0000-0000-00005f5a8609"
       (reference "C1") (unit 1) (value "0.1uF") (footprint "Capacitor_SMD:C_0603_1608Metric")
@@
       (reference "C17") (unit 1) (value "CP") (footprint "Capacitor_SMD:C_1206_3216Metric")
     )
+    (path "/9f4fa5bd-087a-4d9f-a53a-c695f2d95a3c"
+      (reference "D1") (unit 1) (value "LED") (footprint "LED_SMD:LED_0603_1608Metric_Pad1.05x0.95mm_HandSolder")
+    )
     (path "/383a111f-2b69-4da3-91af-c6bc26ff83d1"
       (reference "J1") (unit 1) (value "Conn_01x10_Male") (footprint "Connector_PinHeader_2.54mm:PinHeader_1x10_P2.54mm_Vertical")
@@
       (reference "Q7") (unit 1) (value "BSS138") (footprint "Package_TO_SOT_SMD:SOT-23")
     )
+    (path "/cd5f319f-b5a4-4bea-ac6e-c3375cd7fbb7"
+      (reference "R1") (unit 1) (value "R") (footprint "Resistor_SMD:R_0603_1608Metric_Pad1.05x0.95mm_HandSolder")
+    )
     (path "/ca4496b2-72ae-4f01-a82b-f9c1ef4a576d"
